Commit message: gazebo topics unified for simplicity.

File: simulation/surenaV_description/urdf/surenaV.urdf (robot description, URDF)
Before this commit: robot surenaV, 33 links, 32 joints
Joints:
- joint head_roll_joint: axis -1 0 0 -> 1 0 0
- joint l_arm_pitch_joint: axis 0 -1 0 -> 0 1 0
- joint l_forearm_link_joint: axis 0 0 1 -> 0 0 -1
- joint l_forearm_roll_joint: axis 0 -1 0 -> 0 1 0
- joint l_hand_roll_joint: axis 0 -1 0 -> 0 1 0
- joint r_arm_pitch_joint: axis 0 -1 0 -> 0 1 0
- joint r_arm_roll_joint: axis -1 0 0 -> 1 0 0
- joint r_elbow_pitch_joint: axis 0 0 -1 -> 0 0 1
- joint r_forearm_link_joint: axis 0 0 -1 -> 0 0 1
- joint r_forearm_roll_joint: axis 0 -1 0 -> 0 1 0
- joint r_hand_pitch_joint: axis -1 0 0 -> 0 -1 0
- joint r_hand_roll_joint: axis 0 -1 0 -> 1 0 0

Commit message: fix hands and legs axis on simulation

File: simulation/surenaV_description/urdf/surenaV.urdf (robot description, URDF)
Before this commit: robot surenaV, 33 links, 32 joints
Joints:
- joint l_forearm_link_joint: origin xyz=0 0.03075 -0.07083 rpy=0 0 0 -> xyz=0 0.03075 -0.07083 rpy=0 0 1.57
- joint l_hand_pitch_joint: axis 1 0 0 -> 0 -1 0
- joint l_hand_roll_joint: axis 0 1 0 -> 1 0 0
- joint r_forearm_link_joint: origin xyz=0 -0.03075 -0.07083 rpy=0 0 0 -> xyz=0 -0.03075 -0.07083 rpy=0 0 -1.57
